File: antController.kicad_sch (KiCad schematic)
At the start: 63 parts, among them J1 Lichtenprog_conn, J2 IDC10, J3 PWRINS, J4 FRONT_PANEL, J5 SMA CONN, Q1 MMBT3904, Q2 MMBT3904, SW1 B_RST, SW2 B1/BOOT, SW3 B2, SW4 B3, SW5 B3, U1 PCA9306DC, U2 ESP32-WROOM-32U, U3 AZ1117-3.3, U4 LM317_TO-220

Commit message: finish routing and silk
Connections:
- net +VDC: now also R18.2; no longer D4.2 (A)
- net GND: now also D4.1 (K); no longer R18.1
- new net: D4.2 (A), R18.1
Other:
- moved on the sheet: D4, R18
Changed lines of the file:
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@@
 (kicad_sch (version 20211123) (generator eeschema)
   (paper "A4")
-  (junction (at 83.82 109.22) (diameter 0) (color 0 0 0 0)
-  )
   (junction (at 187.96 133.35) (diameter 0) (color 0 0 0 0)
   )
@@
     (stroke (width 0) (type default) (color 0 0 0 0))
   )
-  (bus (pts (xy 83.82 92.71) (xy 83.82 109.22))
-    (stroke (width 0) (type default) (color 0 0 0 0))
-  )
   (wire (pts (xy 33.02 46.99) (xy 41.91 46.99))
     (stroke (width 0) (type default) (color 0 0 0 0))
@@
     (stroke (width 0) (type default) (color 0 0 0 0))
   )
-  (bus (pts (xy 83.82 109.22) (xy 170.18 109.22))
-    (stroke (width 0) (type default) (color 0 0 0 0))
-  )
   (wire (pts (xy 261.62 67.31) (xy 265.43 67.31))
     (stroke (width 0) (type default) (color 0 0 0 0))
@@
     (stroke (width 0) (type default) (color 0 0 0 0))
   )
-  (bus (pts (xy 55.88 109.22) (xy 83.82 109.22))
-    (stroke (width 0) (type default) (color 0 0 0 0))
-  )
   (wire (pts (xy 46.99 19.05) (xy 46.99 24.13))
     (stroke (width 0) (type default) (color 0 0 0 0))
@@
     (stroke (width 0) (type default) (color 0 0 0 0))
   )
-  (bus (pts (xy 170.18 101.6) (xy 170.18 109.22))
-    (stroke (width 0) (type default) (color 0 0 0 0))
-  )
   (wire (pts (xy 63.5 19.05) (xy 66.04 19.05))
     (stroke (width 0) (type default) (color 0 0 0 0))
@@
     (pin "8")
   )
-  (symbol (lib_id "Device:R") (at 35.56 162.56 0) (mirror x) (unit 1)
+  (symbol (lib_id "Device:R") (at 35.56 152.4 0) (mirror x) (unit 1)
     (in_bom yes) (on_board yes)
-    (property "Reference" "R18" (id 0) (at 33.782 161.3916 0)
+    (property "Reference" "R18" (id 0) (at 33.782 151.2316 0)
       (effects (font (size 1.27 1.27)) (justify right))
     )
-    (property "Value" "100k" (id 1) (at 33.782 163.703 0)
+    (property "Value" "100k" (id 1) (at 33.782 153.543 0)
       (effects (font (size 1.27 1.27)) (justify right))
     )
-    (property "Footprint" "Resistor_SMD:R_0402_1005Metric" (id 2) (at 33.782 162.56 90)
+    (property "Footprint" "Resistor_SMD:R_0402_1005Metric" (id 2) (at 33.782 152.4 90)
       (effects (font (size 1.27 1.27)) hide)
     )
-    (property "Datasheet" "~" (id 3) (at 35.56 162.56 0)
+    (property "Datasheet" "~" (id 3) (at 35.56 152.4 0)
       (effects (font (size 1.27 1.27)) hide)
     )
@@
     (pin "1")
   )
-  (symbol (lib_id "Device:LED") (at 35.56 152.4 270) (mirror x) (unit 1)
+  (symbol (lib_id "Device:LED") (at 35.56 162.56 270) (mirror x) (unit 1)
     (in_bom yes) (on_board yes)
-    (property "Reference" "D4" (id 0) (at 32.5628 151.4094 90)
+    (property "Reference" "D4" (id 0) (at 32.5628 161.5694 90)
       (effects (font (size 1.27 1.27)) (justify right))
     )
-    (property "Value" "LED_RED" (id 1) (at 32.5628 153.7208 90)
+    (property "Value" "LED_RED" (id 1) (at 32.5628 163.8808 90)
       (effects (font (size 1.27 1.27)) (justify right))
     )
-    (property "Footprint" "LED_SMD:LED_0603_1608Metric" (id 2) (at 35.56 152.4 0)
+    (property "Footprint" "LED_SMD:LED_0603_1608Metric" (id 2) (at 35.56 162.56 0)
       (effects (font (size 1.27 1.27)) hide)
     )
-    (property "Datasheet" "~" (id 3) (at 35.56 152.4 0)
+    (property "Datasheet" "~" (id 3) (at 35.56 162.56 0)
       (effects (font (size 1.27 1.27)) hide)
     )
@@
       (reference "#PWR0128") (unit 1) (value "GND2") (footprint "")
     )
-    (path "/ea3a19db-d722-4aea-937e-ab71ca8d288d/2314dcfe-36c4-4cfe-af2c-e540b210abc2"
-      (reference "#PWR0129") (unit 1) (value "GND") (footprint "")
+    (path "/ea3a19db-d722-4aea-937e-ab71ca8d288d/ab34314b-ee59-42db-a2a5-71d99e0cfab2"
+      (reference "#PWR0129") (unit 1) (value "GND2") (footprint "")
     )
     (path "/ea3a19db-d722-4aea-937e-ab71ca8d288d/0738411b-00b9-4204-816c-236c1eff344f"
@@
       (reference "#PWR0132") (unit 1) (value "+3V3") (footprint "")
     )
-    (path "/ea3a19db-d722-4aea-937e-ab71ca8d288d/65fbe17c-935e-4397-a51a-b7d88ab62f32"
-      (reference "#PWR0133") (unit 1) (value "+5V") (footprint "")
+    (path "/ea3a19db-d722-4aea-937e-ab71ca8d288d/dab6095c-a70f-4718-87b9-7830045c5991"
+      (reference "#PWR0133") (unit 1) (value "+5VD") (footprint "")
     )
     (path "/ea3a19db-d722-4aea-937e-ab71ca8d288d/cc9dd56b-88ad-497b-b308-d80dbf3f962c"
@@
       (reference "#PWR0198") (unit 1) (value "GND2") (footprint "")
     )
+    (path "/ea3a19db-d722-4aea-937e-ab71ca8d288d/9ce8c060-ebf1-4a7d-b3bb-6ac8ee9c8c94"
+      (reference "#PWR0199") (unit 1) (value "+3V3") (footprint "")
+    )
+    (path "/ea3a19db-d722-4aea-937e-ab71ca8d288d/4c9626ac-c7a7-458a-94d5-be153eb7d837"
+      (reference "#PWR0200") (unit 1) (value "GND") (footprint "")
+    )
     (path "/757d1244-fc3b-4ccd-83d9-51daecebb46f"

Commit message: prod files
Parts:
- removed J3: PWRINS, TerminalBlock_MetzConnect:TerminalBlock_MetzConnect_Type055_RT01504HDWU_1x04_P5.00mm_Horizontal, symbol Connector:Screw_Terminal_01x04
- added C57: 220u, Capacitor_THT:CP_Radial_D8.0mm_P3.50mm, symbol Device:C_Polarized
- added J15, J16, J17, J3: VIN, Critbit_lib:DG235-5.0, symbol Connector:Screw_Terminal_01x01
Connections:
- net +5V: now also C57.1
- net +VDC: now also J16.1 (Pin_1)
- net 5V_IN: now also J3.1 (Pin_1)
- net GND: now also C57.2, J15.1 (Pin_1), J17.1 (Pin_1)
Other:
- moved on the sheet: D1, R13

Commit message: PoC API call for IO
Other:
- note added: "Rev 1.0 - Initial release Rev 1.1 TODO: - I2C and TX/RX are swapped on connectors - More space for LM317 radiator - Screw holes too close to the edge - Button descriptors on silk - Fix BOM / PnP files (capacitor errors)"
- note removed: "Wymagania 15. Oszacuj pobór prądów 3,3/5V, w razie czego miejsce na radiatory dla stabilizatorów. Policzyć rezystory. 2. BUZ11 TO220, dren w środku 4. drugi PCA steruje 16-toma przekaźnikami (wg. pin-outu przesłanego) poprzez tranzystory bipolarne 5. trzeci PCA dolna ósemka - transoptory, rezystor szeregowy diody 4k7 6. 12 wejść zabezpieczyc filtrem RF R=10k + C=10nF Gniazda DB25 na jednaj krawęd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"
Changed lines of the file:
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@@
     (effects (font (size 1.27 1.27)) (justify left bottom))
   )
-  (text "Wymagania\n\n\n15. Oszacuj pobór prądów 3,3/5V, w razie czego miejsce na radiatory dla stabilizatorów. Policzyć rezystory. \n\n2. BUZ11 TO220, dren w środku\n\n4. drugi PCA steruje 16-toma przekaźnikami (wg. pin-outu przesłanego) poprzez tranzystory bipolarne\n\n5. trzeci PCA dolna ósemka - transoptory, rezystor szeregowy diody 4k7\n\n6. 12 wejść zabezpieczyc filtrem RF R=10k + C=10nF\n\nGniazda DB25 na jednaj krawędzi:\n\nJ1:  Sink1-16 (16pin) + masa (5 pin) + VD (2 pin koło siebie z 100n+1n) + 15V (2 pin koło siebie z 100n+1n)\n\nJ2: 12x styki przekaźników (24 pin) + masa. Pozostałe 4 przekaźniki pozostawimy niepodłączone do gniazd, tylko goldpiny jako zapasowe, np. do podłączenia z J4\n\nJ3: BUFF1-8 + masa cyfrowa + 5V (8pin), 8 wyjść opto (16 pin), masa\n\nJ4: 3x4 wejścia + masy cyfrowe (15 pin) , masa (2 pin), pozostałe 8 pin goldpiny jako zapasowe"
-    (at 297.18 170.18 0)
+  (text "Rev 1.0\n- Initial release\nRev 1.1\nTODO:\n- I2C and TX/RX are swapped on connectors\n- More space for LM317 radiator\n- Screw holes too close to the edge\n- Button descriptors on silk\n- Fix BOM / PnP files (capacitor errors)\n"
+    (at 232.41 124.46 0)
     (effects (font (size 1.27 1.27)) (justify left bottom))
   )
