File: antController.kicad_sch (KiCad schematic)
At the start: 67 parts, among them J1 Lichtenprog_conn, J15 VIN, J16 VIN, J17 VIN, J2 IDC10, J3 VIN, J4 FRONT_PANEL, J5 SMA CONN, Q1 MMBT3904, Q2 MMBT3904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

Commit message: from future import missing resistors
Other:
- note added: "Rev 1.0 - Initial release Rev 1.1 TODO: - I2C and TX/RX are swapped on connectors between boards - More space for LM317 radiator - Screw holes too close to the edge - Terminal screws inaccesible after assembly - Button descriptors on silk - Fix BOM / PnP files (capacitor errors) - DTR/RTS lines must not have C filters, only RC is allowed - Add pads to all outputs for manual rework DONE: - Added p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"
- note removed: "Rev 1.0 - Initial release Rev 1.1 TODO: - I2C and TX/RX are swapped on connectors - More space for LM317 radiator - Screw holes too close to the edge - Button descriptors on silk - Fix BOM / PnP files (capacitor errors) - DTR/RTS lines must not have C filters, only RC is allowed"
