File: optocoupler.kicad_sch (KiCad schematic)
At the start: 4 parts, among them U18 LTV-356T

Commit message: routing mostly done, fixing schematic issues
Parts:
- D29: renamed from D5; value LED -> LED_RED; footprint Diode_SMD:D_0603_1608Metric -> LED_SMD:LED_0603_1608Metric
- R131: renamed from R107; value 10k -> 33k
Changed lines of the file:
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@@
   (symbol (lib_id "Device:R") (at 36.83 35.56 0) (mirror x) (unit 1)
     (in_bom yes) (on_board yes)
-    (property "Reference" "R107" (id 0) (at 35.052 34.3916 0)
+    (property "Reference" "R131" (id 0) (at 35.052 34.3916 0)
       (effects (font (size 1.27 1.27)) (justify right))
     )
-    (property "Value" "10k" (id 1) (at 35.56 36.83 0)
+    (property "Value" "33k" (id 1) (at 35.56 36.83 0)
       (effects (font (size 1.27 1.27)) (justify right))
     )
@@
   (symbol (lib_id "Device:LED") (at 36.83 26.67 270) (mirror x) (unit 1)
     (in_bom yes) (on_board yes) (fields_autoplaced)
-    (property "Reference" "D5" (id 0) (at 33.909 27.4228 90)
+    (property "Reference" "D29" (id 0) (at 33.909 27.4228 90)
       (effects (font (size 1.27 1.27)) (justify right))
     )
-    (property "Value" "LED" (id 1) (at 33.909 29.9597 90)
+    (property "Value" "LED_RED" (id 1) (at 33.909 29.9597 90)
       (effects (font (size 1.27 1.27)) (justify right))
     )
-    (property "Footprint" "Diode_SMD:D_0603_1608Metric" (id 2) (at 36.83 26.67 0)
+    (property "Footprint" "LED_SMD:LED_0603_1608Metric" (id 2) (at 36.83 26.67 0)
       (effects (font (size 1.27 1.27)) hide)
     )
