File: relay.kicad_sch (KiCad schematic)
At the start: 6 parts, among them K1 G5V-1, Q19 2N7002

Commit message: routing mostly done, fixing schematic issues
Parts:
- removed Q19: 2N7002, Package_TO_SOT_SMD:SOT-23, symbol Transistor_FET:2N7002
- added D44: 1N4148WS, Diode_SMD:D_SOD-323, symbol Diode:1N4148WS
- added Q19: MMBT3904, Package_TO_SOT_SMD:SOT-23, symbol Transistor_BJT:MMBT3904
- D22: value LED -> LED_RED; footprint Diode_SMD:D_0603_1608Metric -> LED_SMD:LED_0603_1608Metric
- R124: value 10k -> 33k
Connections:
- net GND: now also Q19.2 (E)
- net VCOIL: now also D44.1 (K)
- net at R70.1, R71.2: now also Q19.1 (B)
- net at K1.9: now also D44.2 (A), Q19.3 (C)
Changed lines of the file:
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@@
   (junction (at 111.76 120.65) (diameter 0) (color 0 0 0 0)
+  )
+  (junction (at 121.92 90.17) (diameter 0) (color 0 0 0 0)
+  )
+  (junction (at 109.22 64.77) (diameter 0) (color 0 0 0 0)
   )
   (junction (at 111.76 99.06) (diameter 0) (color 0 0 0 0)
@@
     (stroke (width 0) (type default) (color 0 0 0 0))
   )
-  (wire (pts (xy 121.92 83.82) (xy 121.92 93.98))
+  (wire (pts (xy 121.92 83.82) (xy 121.92 90.17))
     (stroke (width 0) (type default) (color 0 0 0 0))
   )
@@
     (stroke (width 0) (type default) (color 0 0 0 0))
   )
+  (wire (pts (xy 121.92 90.17) (xy 121.92 93.98))
+    (stroke (width 0) (type default) (color 0 0 0 0))
+  )
   (wire (pts (xy 111.76 113.03) (xy 111.76 120.65))
     (stroke (width 0) (type default) (color 0 0 0 0))
   )
+  (wire (pts (xy 109.22 64.77) (xy 109.22 72.39))
+    (stroke (width 0) (type default) (color 0 0 0 0))
+  )
   (wire (pts (xy 134.62 68.58) (xy 139.7 68.58))
     (stroke (width 0) (type default) (color 0 0 0 0))
@@
     (stroke (width 0) (type default) (color 0 0 0 0))
   )
+  (wire (pts (xy 109.22 64.77) (xy 86.36 64.77))
+    (stroke (width 0) (type default) (color 0 0 0 0))
+  )
   (wire (pts (xy 95.25 107.95) (xy 95.25 109.22))
     (stroke (width 0) (type default) (color 0 0 0 0))
@@
     (stroke (width 0) (type default) (color 0 0 0 0))
   )
-  (wire (pts (xy 121.92 64.77) (xy 86.36 64.77))
+  (wire (pts (xy 121.92 64.77) (xy 109.22 64.77))
     (stroke (width 0) (type default) (color 0 0 0 0))
   )
@@
     (stroke (width 0) (type default) (color 0 0 0 0))
   )
+  (wire (pts (xy 121.92 90.17) (xy 109.22 90.17))
+    (stroke (width 0) (type default) (color 0 0 0 0))
+  )
+  (wire (pts (xy 109.22 90.17) (xy 109.22 80.01))
+    (stroke (width 0) (type default) (color 0 0 0 0))
+  )
   (wire (pts (xy 111.76 99.06) (xy 114.3 99.06))
     (stroke (width 0) (type default) (color 0 0 0 0))
   )
-  (text "Idc 40mA" (at 114.3 86.36 0)
+  (text "Idc 40mA" (at 111.76 88.9 0)
     (effects (font (size 1.27 1.27)) (justify left bottom))
   )
@@
     (pin "2")
   )
-  (symbol (lib_id "Transistor_FET:2N7002") (at 119.38 99.06 0) (unit 1)
-    (in_bom yes) (on_board yes) (fields_autoplaced)
-    (property "Reference" "Q19" (id 0) (at 124.587 98.2253 0)
-      (effects (font (size 1.27 1.27)) (justify left))
-    )
-    (property "Value" "2N7002" (id 1) (at 124.587 100.7622 0)
-      (effects (font (size 1.27 1.27)) (justify left))
-    )
-    (property "Footprint" "Package_TO_SOT_SMD:SOT-23" (id 2) (at 124.46 100.965 0)
-      (effects (font (size 1.27 1.27) italic) (justify left) hide)
-    )
-    (property "Datasheet" "https://www.onsemi.com/pub/Collateral/NDS7002A-D.PDF" (id 3) (at 119.38 99.06 0)
-      (effects (font (size 1.27 1.27)) (justify left) hide)
-    )
-    (pin "1")
-    (pin "2")
-    (pin "3")
+  (symbol (lib_id "Diode:1N4148WS") (at 109.22 76.2 270) (unit 1)
+    (in_bom yes) (on_board yes)
+    (property "Reference" "D44" (id 0) (at 105.41 74.93 90)
+      (effects (font (size 1.27 1.27)) (justify left))
+    )
+    (property "Value" "1N4148WS" (id 1) (at 96.52 77.47 90)
+      (effects (font (size 1.27 1.27)) (justify left))
+    )
+    (property "Footprint" "Diode_SMD:D_SOD-323" (id 2) (at 104.775 76.2 0)
+      (effects (font (size 1.27 1.27)) hide)
+    )
+    (property "Datasheet" "https://www.vishay.com/docs/85751/1n4148ws.pdf" (id 3) (at 109.22 76.2 0)
+      (effects (font (size 1.27 1.27)) hide)
+    )
+    (pin "1")
+    (pin "2")
   )
   (symbol (lib_id "Relay:G5V-1") (at 127 76.2 0) (unit 1)
@@
       (effects (font (size 1.27 1.27)) (justify left))
     )
-    (property "Value" "LED" (id 1) (at 97.282 107.4297 90)
-      (effects (font (size 1.27 1.27)) (justify left))
-    )
-    (property "Footprint" "Diode_SMD:D_0603_1608Metric" (id 2) (at 95.25 104.14 0)
+    (property "Value" "LED_RED" (id 1) (at 97.282 107.4297 90)
+      (effects (font (size 1.27 1.27)) (justify left))
+    )
+    (property "Footprint" "LED_SMD:LED_0603_1608Metric" (id 2) (at 95.25 104.14 0)
       (effects (font (size 1.27 1.27)) hide)
     )
@@
       (effects (font (size 1.27 1.27)) (justify right))
     )
-    (property "Value" "10k" (id 1) (at 93.98 114.3 0)
+    (property "Value" "33k" (id 1) (at 93.98 114.3 0)
       (effects (font (size 1.27 1.27)) (justify right))
     )
@@
     (pin "2")
   )
+  (symbol (lib_id "Transistor_BJT:MMBT3904") (at 119.38 99.06 0) (unit 1)
+    (in_bom yes) (on_board yes) (fields_autoplaced)
+    (property "Reference" "Q19" (id 0) (at 124.2314 98.2253 0)
+      (effects (font (size 1.27 1.27)) (justify left))
+    )
+    (property "Value" "MMBT3904" (id 1) (at 124.2314 100.7622 0)
+      (effects (font (size 1.27 1.27)) (justify left))
+    )
+    (property "Footprint" "Package_TO_SOT_SMD:SOT-23" (id 2) (at 124.46 100.965 0)
+      (effects (font (size 1.27 1.27) italic) (justify left) hide)
+    )
+    (property "Datasheet" "https://www.onsemi.com/pub/Collateral/2N3903-D.PDF" (id 3) (at 119.38 99.06 0)
+      (effects (font (size 1.27 1.27)) (justify left) hide)
+    )
+    (pin "1")
+    (pin "2")
+    (pin "3")
+  )
 )
